Commit message: Traker 1/2

File: elfin/elfin_description/urdf/elfin3.urdf.xacro (robot description, xacro)
@@ -1,8 +1,12 @@
 <robot
   name="elfin3" xmlns:xacro="http://www.ros.org/wiki/xacro">
+  <xacro:include filename="$(find elfin_description)/urdf/_d435.urdf.xacro"/>
   <xacro:include filename="$(find elfin_description)/urdf/materials.xacro" />
   <xacro:include filename="$(find elfin_description)/urdf/elfin_robot.gazebo" />
   <xacro:include filename="$(find elfin_description)/urdf/elfin_transmission.xacro" />
   <xacro:property name="PI" value="3.1415926535897931"/>
+  <xacro:sensor_d435 name="relasense" parent="elfin_dummy_gripper">
+  <origin xyz="0.04 0 -0.05" rpy="${-PI} ${3*PI/2} 0"/>
+  </xacro:sensor_d435>
   <link name="world"/>
   <joint name="world_base" type="fixed">

Commit message: Near traking

File: elfin/elfin_description/urdf/elfin3.urdf.xacro (robot description, xacro)
@@ -6,7 +6,4 @@
   <xacro:include filename="$(find elfin_description)/urdf/elfin_transmission.xacro" />
   <xacro:property name="PI" value="3.1415926535897931"/>
-  <xacro:sensor_d435 name="relasense" parent="elfin_dummy_gripper">
-  <origin xyz="0.04 0 -0.05" rpy="${-PI} ${3*PI/2} 0"/>
-  </xacro:sensor_d435>
   <link name="world"/>
   <joint name="world_base" type="fixed">
@@ -434,3 +431,6 @@
       link="elfin_dummy_gripper" />
   </joint>
+  <xacro:sensor_d435 name="relasense" parent="elfin_dummy_gripper">
+    <origin xyz="0.04 0 -0.05" rpy="${-PI} ${3*PI/2} 0"/>
+  </xacro:sensor_d435>
 </robot>

Commit message: Inizio finale

File: elfin/elfin_description/urdf/elfin3.urdf.xacro (robot description, xacro)
@@ -432,5 +432,5 @@
   </joint>
   <xacro:sensor_d435 name="relasense" parent="elfin_dummy_gripper">
-    <origin xyz="0.04 0 -0.05" rpy="${-PI} ${3*PI/2} 0"/>
+    <origin xyz="0.0 0.0 -0.002" rpy="${0} ${3*PI/2} 0"/>
   </xacro:sensor_d435>
 </robot>

File: elfin/elfin_description/urdf/elfin3_experiment1.urdf.xacro (robot description, xacro)
@@ -2,4 +2,5 @@
   name="elfin3" xmlns:xacro="http://www.ros.org/wiki/xacro">
   <xacro:include filename="$(find elfin_description)/urdf/materials.xacro" />
+  <xacro:include filename="$(find elfin_description)/urdf/_d435.urdf.xacro"/>
   <xacro:include filename="$(find elfin_description)/urdf/elfin_robot_experiment1.gazebo" />
   <xacro:include filename="$(find elfin_description)/urdf/elfin_transmission_experiment1.xacro" />
@@ -488,3 +489,6 @@
     <origin xyz="0 -0.04 0" rpy="0 0 0" />
   </joint>
+  <xacro:sensor_d435 name="relasense" parent="elfin_link6">
+    <origin xyz="0.0 -0.091 0.0" rpy="0 0 ${-PI/2}"/>
+  </xacro:sensor_d435>
 </robot>

Commit message: Going to point

File: elfin/elfin_description/urdf/elfin3.urdf.xacro (robot description, xacro)
@@ -432,5 +432,5 @@
   </joint>
   <xacro:sensor_d435 name="relasense" parent="elfin_dummy_gripper">
-    <origin xyz="0.0 0.0 -0.002" rpy="${0} ${3*PI/2} 0"/>
+    <origin xyz="0.04 0.0 -0.05" rpy="${-PI} ${3*PI/2} 0"/>
   </xacro:sensor_d435>
 </robot>
